Commit message: not working again

File: final_assignment/urdf/robot_assignment.xacro (robot description, xacro)
@@ -1,9 +1,11 @@
 <?xml version="1.0" ?>
-<robot name="m2wr" xmlns:xacro="https://www.ros.org/wiki/xacro" >
-  <xacro:include filename="$(find inspection_robot)/urdf/materials.xacro" />
-  <xacro:include filename="$(find inspection_robot)/urdf/robot_assignment.gazebo" />
+<robot name="robot_assignment" xmlns:xacro="https://www.ros.org/wiki/xacro">
+  <xacro:include filename="$(find final_assignment)/urdf/materials.xacro" />
+  <xacro:include filename="$(find final_assignment)/urdf/robot_assignment.gazebo" />
   <xacro:macro name="cylinder_inertia" params="mass r l">
-    <inertia ixx="${mass*(3*r*r+l*l)/12}" ixy = "0" ixz = "0"
-    iyy="${mass*(3*r*r+l*l)/12}" iyz = "0" izz="${mass*(r*r)/2}" />
+    <inertia
+      ixx="${mass*(3*r*r+l*l)/12}" ixy = "0" ixz = "0"
+      iyy="${mass*(3*r*r+l*l)/12}" iyz = "0" izz="${mass*(r*r)/2}"
+    />
   </xacro:macro>
   <xacro:macro name="link_wheel" params="name">
@@ -28,5 +30,5 @@
     </link>
   </xacro:macro>
-  <xacro:macro name="arm_link" params="name arm_link_length xyz_origin">
+  <xacro:macro name="link_arm" params="name length xyz_origin">
 		<link name="${name}">
 			<inertial>
@@ -38,5 +40,5 @@
 				<origin rpy="0 0 0" xyz="${xyz_origin}"/>
         <geometry>
-          <cylinder length="${arm_link_length}" radius="0.04"/>
+          <cylinder length="${length}" radius="0.04"/>
         </geometry>
 			</collision>
@@ -44,5 +46,5 @@
 				<origin rpy="0 0 0" xyz="${xyz_origin}"/>
         <geometry>
-          <cylinder length="${arm_link_length}" radius="0.04"/>
+          <cylinder length="${length}" radius="0.04"/>
         </geometry>
 			</visual>
@@ -59,5 +61,5 @@
     </joint>
   </xacro:macro>
-  <xacro:macro name="revolute_joint" params="name parent child origin_xyz axis_xyz">
+  <xacro:macro name="joint_arm" params="name parent child origin_xyz axis_xyz">
     <joint name="${name}" type="revolute">
       <axis xyz="${axis_xyz}"/>
@@ -66,8 +68,9 @@
       <parent link="${parent}"/>
       <child link="${child}"/>
-    </joint>
-  </xacro:macro>
+      <joint_properties damping="1.0" friction="1.0"/>
+    </joint>
+  </xacro:macro>
+  <!-- MAIN BODY -->
   <link name="base_link">
-    <!-- pose and inertial -->
     <pose>0 0 0.1 0 0 0</pose>
     <inertial>
@@ -76,4 +79,5 @@
       <inertia ixx="0.0395416666667" ixy="0" ixz="0" iyy="0.106208333333" iyz="0" izz="0.106208333333"/>
     </inertial>
+    <!-- CHASSIS -->
     <collision name="collision_chassis">
       <geometry>
@@ -88,5 +92,5 @@
       <material name="blue"/>
     </visual>
-      <!-- caster front -->
+    <!-- CASTER FRONT -->
     <collision name="caster_front_collision">
       <origin rpy=" 0 0 0" xyz="0.35 0 -0.05"/>
@@ -112,9 +116,11 @@
     </visual>
   </link>
-  <!-- Create wheels -->
+  <!-- WHEEL RIGHT -->
   <xacro:link_wheel name="link_right_wheel" />
+  <xacro:joint_wheel name="joint_right_wheel"  child="link_right_wheel"  origin_xyz="-0.05 0.15 0"  />
+  <!-- WHEEL LEFT -->
   <xacro:link_wheel name="link_left_wheel" />
-  <xacro:joint_wheel name="joint_right_wheel"  child="link_right_wheel"  origin_xyz="-0.05 0.15 0"  />
   <xacro:joint_wheel name="joint_left_wheel"   child="link_left_wheel"   origin_xyz="-0.05 -0.15 0"  />
+  <!-- LASER -->
   <link name="laser">
     <inertial>
@@ -142,5 +148,5 @@
     <child link="laser"/>
   </joint>
-<!--arm definition -->
+  <!-- ARM BASE LINK -->
   <link name="arm_base_link">
   	<inertial>
@@ -168,11 +174,15 @@
   	<child link="arm_base_link"/>
   </joint>
-  <xacro:arm_link name="arm_link_01" arm_link_length="0.15" xyz_origin="0 0 0.075"/>
-  <xacro:arm_link name="arm_link_02" arm_link_length="0.15" xyz_origin="0 0 0.075"/>
-  <xacro:arm_link name="arm_link_03" arm_link_length="0.06" xyz_origin="0 0 0.03"/>
-  <xacro:revolute_joint name="arm_joint_01" child="arm_link_01" parent="arm_base_link" origin_xyz="0 0 0.025" axis_xyz="0 0 1"/>
-  <xacro:revolute_joint name="arm_joint_02" child="arm_link_02" parent="arm_link_01" origin_xyz="0 0 0.15" axis_xyz="1 0 0"/>
-  <xacro:revolute_joint name="arm_joint_03" child="arm_link_03" parent="arm_link_02" origin_xyz="0 0 0.15" axis_xyz="0 1 0"/>
-    <link name="camera_link">
+  <!-- ARM 0 -->
+  <xacro:link_arm name="arm_link_01" length="0.15" xyz_origin="0 0 0.075"/>
+  <xacro:joint_arm name="arm_joint_01" child="arm_link_01" parent="arm_base_link" origin_xyz="0 0 0.025" axis_xyz="0 0 1"/>
+  <!-- ARM 1 -->
+  <xacro:link_arm name="arm_link_02" length="0.15" xyz_origin="0 0 0.075"/>
+  <xacro:joint_arm name="arm_joint_02" child="arm_link_02" parent="arm_link_01" origin_xyz="0 0 0.15" axis_xyz="1 0 0"/>
+  <!-- ARM 2 -->
+  <xacro:link_arm name="arm_link_03" length="0.06" xyz_origin="0 0 0.03"/>
+  <xacro:joint_arm name="arm_joint_03" child="arm_link_03" parent="arm_link_02" origin_xyz="0 0 0.15" axis_xyz="0 1 0"/>
+  <!-- CAMERA -->
+  <link name="camera_link">
   	<inertial>
   		<mass value="0.025"/>
@@ -201,33 +211,34 @@
   	<child link="camera_link"/>
   </joint>
-<transmission name="arm_joint_01_trans">
-	<type>transmission_interface/SimpleTransmission</type>
-	<joint name="arm_joint_01">
-		<hardwareInterface>hardware_interface/EffortJointInterface</hardwareInterface>
-	</joint>
-	<actuator name="motor1">
-		<hardwareInterface>hardware_interface/EffortJointInterface</hardwareInterface>
-		<mechanicalInterface>1</mechanicalInterface>
-	</actuator>
-</transmission>
-<transmission name="arm_joint_02_trans">
-	<type>transmission_interface/SimpleTransmission</type>
-	<joint name="arm_joint_02">
-		<hardwareInterface>hardware_interface/EffortJointInterface</hardwareInterface>
-	</joint>
-	<actuator name="motor2">
-		<hardwareInterface>hardware_interface/EffortJointInterface</hardwareInterface>
-		<mechanicalInterface>1</mechanicalInterface>
-	</actuator>
-</transmission>
-<transmission name="arm_joint_03_trans">
-	<type>transmission_interface/SimpleTransmission</type>
-	<joint name="arm_joint_03">
-		<hardwareInterface>hardware_interface/EffortJointInterface</hardwareInterface>
-	</joint>
-	<actuator name="motor3">
-		<hardwareInterface>hardware_interface/EffortJointInterface</hardwareInterface>
-		<mechanicalInterface>1</mechanicalInterface>
-	</actuator>
-</transmission>
+  <!-- TRANSMISSION -->
+  <transmission name="arm_joint_01_trans">
+    <type>transmission_interface/SimpleTransmission</type>
+    <joint name="arm_joint_01">
+      <hardwareInterface>hardware_interface/EffortJointInterface</hardwareInterface>
+    </joint>
+    <actuator name="motor1">
+      <hardwareInterface>hardware_interface/EffortJointInterface</hardwareInterface>
+      <mechanicalInterface>1</mechanicalInterface>
+    </actuator>
+  </transmission>
+  <transmission name="arm_joint_02_trans">
+    <type>transmission_interface/SimpleTransmission</type>
+    <joint name="arm_joint_02">
+      <hardwareInterface>hardware_interface/EffortJointInterface</hardwareInterface>
+    </joint>
+    <actuator name="motor2">
+      <hardwareInterface>hardware_interface/EffortJointInterface</hardwareInterface>
+      <mechanicalInterface>1</mechanicalInterface>
+    </actuator>
+  </transmission>
+  <transmission name="arm_joint_03_trans">
+    <type>transmission_interface/SimpleTransmission</type>
+    <joint name="arm_joint_03">
+      <hardwareInterface>hardware_interface/EffortJointInterface</hardwareInterface>
+    </joint>
+    <actuator name="motor3">
+      <hardwareInterface>hardware_interface/EffortJointInterface</hardwareInterface>
+      <mechanicalInterface>1</mechanicalInterface>
+    </actuator>
+  </transmission>
 </robot>
