Commit message: urdf

File: final_assignment/urdf/robot.xacro (robot description, xacro)
@@ -138,5 +138,5 @@
       <origin rpy="0 0 0" xyz="0 0 0"/>
       <geometry>
-        <box size="0.08 0.08 0.08"/>
+        <box size="0.10 0.10 0.10"/>
       </geometry>
       <material name="green"/>
@@ -166,5 +166,5 @@
       <origin rpy="0 0 0" xyz="0 0 0.15"/>
       <geometry>
-        <box size="0.05 0.05 0.2"/>
+        <box size="0.05 0.05 0.3"/>
       </geometry>
       <material name="green"/>
